File: Alimentacion_12v/Alimentacion_12v.sch (KiCad schematic (older format))
At the start: 22 parts, among them J1 USB_B_Micro, J2 Conn_01x02_Male, J3 Conn_01x02_Male, J4 Conn_01x02_Male, J5 Conn_01x03_Female, J6 Conn_01x02_Male, U1 lm2577t-15_NOPB, U2 LM317L_TO92

Commit message: Placa de 12 Voltios V.0.5
Parts:
- removed J1: USB_B_Micro, Connector_USB:USB_Micro-B_Wuerth_614105150721_Vertical_CircularHoles, symbol Connector:USB_B_Micro
- added J1: USB_B, Connector_USB:USB_B_OST_USB-B1HSxx_Horizontal, symbol Connector:USB_B
- C1: footprint Capacitor_THT:C_Disc_D3.0mm_W2.0mm_P2.50mm -> Capacitor_THT:C_Disc_D5.0mm_W2.5mm_P2.50mm
- C2: footprint Capacitor_THT:CP_Radial_D10.0mm_P5.00mm -> Capacitor_THT:CP_Radial_D7.5mm_P2.50mm
- C4: footprint Capacitor_THT:CP_Radial_D10.0mm_P5.00mm -> Capacitor_THT:C_Disc_D3.8mm_W2.6mm_P2.50mm
- C5: footprint Capacitor_THT:C_Disc_D3.0mm_W2.0mm_P2.50mm -> Capacitor_THT:C_Disc_D3.8mm_W2.6mm_P2.50mm
- D1, D2: footprint Diode_THT:D_DO-34_SOD68_P7.62mm_Horizontal -> Diode_THT:D_DO-15_P15.24mm_Horizontal
- U1: footprint LM2577:lm2577t-15&slash_NOPB -> Package_TO_SOT_THT:TO-220-5_P3.4x3.7mm_StaggerEven_Lead3.8mm_Vertical
- U2: footprint Package_TO_SOT_THT:TO-92_Inline -> Package_TO_SOT_THT:TO-220-3_Vertical
Changed lines of the file:
@@
 EESchema Schematic File Version 4
+LIBS:Alimentacion_12v-cache
 EELAYER 26 0
 EELAYER END
@@
 F 0 "U1" H 5800 3537 60  0000 C CNN
 F 1 "lm2577t-15_NOPB" H 5800 3431 60  0000 C CNN
-F 2 "LM2577:lm2577t-15&slash_NOPB" H 5800 3390 60  0001 C CNN
+F 2 "Package_TO_SOT_THT:TO-220-5_P3.4x3.7mm_StaggerEven_Lead3.8mm_Vertical" H 5800 3390 60  0001 C CNN
 F 3 "" H 4700 3150 60  0000 C CNN
 	1    4700 3150
@@
 F 0 "C1" H 4415 3846 50  0000 L CNN
 F 1 "330nF" H 4415 3755 50  0000 L CNN
-F 2 "Capacitor_THT:C_Disc_D3.0mm_W2.0mm_P2.50mm" H 4338 3650 50  0001 C CNN
+F 2 "Capacitor_THT:C_Disc_D5.0mm_W2.5mm_P2.50mm" H 4338 3650 50  0001 C CNN
 F 3 "~" H 4300 3800 50  0001 C CNN
 	1    4300 3800
@@
 F 0 "D2" H 4450 2484 50  0000 C CNN
 F 1 "1N5822" H 4450 2575 50  0000 C CNN
-F 2 "Diode_THT:D_DO-34_SOD68_P7.62mm_Horizontal" H 4450 2525 50  0001 C CNN
+F 2 "Diode_THT:D_DO-15_P15.24mm_Horizontal" H 4450 2525 50  0001 C CNN
 F 3 "http://www.vishay.com/docs/88526/1n5820.pdf" H 4450 2700 50  0001 C CNN
 	1    4450 2700
 	-1   0    0    1
-$EndComp
-$Comp
-L Connector:USB_B_Micro J1
-U 1 1 5C9120E9
-P 2750 3200
-F 0 "J1" H 2805 3667 50  0000 C CNN
-F 1 "USB_B_Micro" H 2805 3576 50  0000 C CNN
-F 2 "Connector_USB:USB_Micro-B_Wuerth_614105150721_Vertical_CircularHoles" H 2900 3150 50  0001 C CNN
-F 3 "~" H 2900 3150 50  0001 C CNN
-	1    2750 3200
-	1    0    0    -1
 $EndComp
 $Comp
@@
 F 0 "C4" H 5185 2454 50  0000 R CNN
 F 1 "0.1uF" H 5185 2545 50  0000 R CNN
-F 2 "Capacitor_THT:CP_Radial_D10.0mm_P5.00mm" H 5338 2350 50  0001 C CNN
+F 2 "Capacitor_THT:C_Disc_D3.8mm_W2.6mm_P2.50mm" H 5338 2350 50  0001 C CNN
 F 3 "~" H 5300 2500 50  0001 C CNN
 	1    5300 2500
@@
 F 0 "D1" H 3400 1884 50  0000 C CNN
 F 1 "1N5822" H 3400 1975 50  0000 C CNN
-F 2 "Diode_THT:D_DO-34_SOD68_P7.62mm_Horizontal" H 3400 1925 50  0001 C CNN
+F 2 "Diode_THT:D_DO-15_P15.24mm_Horizontal" H 3400 1925 50  0001 C CNN
 F 3 "http://www.vishay.com/docs/88526/1n5820.pdf" H 3400 2100 50  0001 C CNN
 	1    3400 2100
@@
 F 0 "U2" H 5450 4992 50  0000 C CNN
 F 1 "LM317L_TO92" H 5450 4901 50  0000 C CNN
-F 2 "Package_TO_SOT_THT:TO-92_Inline" H 5450 4975 50  0001 C CIN
+F 2 "Package_TO_SOT_THT:TO-220-3_Vertical" H 5450 4975 50  0001 C CIN
 F 3 "http://www.ti.com/lit/ds/snvs775k/snvs775k.pdf" H 5450 4750 50  0001 C CNN
 	1    5450 4750
@@
 F 0 "C2" H 4915 5096 50  0000 L CNN
 F 1 "10uF" H 4915 5005 50  0000 L CNN
-F 2 "Capacitor_THT:CP_Radial_D10.0mm_P5.00mm" H 4838 4900 50  0001 C CNN
+F 2 "Capacitor_THT:CP_Radial_D7.5mm_P2.50mm" H 4838 4900 50  0001 C CNN
 F 3 "~" H 4800 5050 50  0001 C CNN
 	1    4800 5050
@@
 F 0 "C5" H 6315 5046 50  0000 L CNN
 F 1 "100nF" H 6315 4955 50  0000 L CNN
-F 2 "Capacitor_THT:C_Disc_D3.0mm_W2.0mm_P2.50mm" H 6238 4850 50  0001 C CNN
+F 2 "Capacitor_THT:C_Disc_D3.8mm_W2.6mm_P2.50mm" H 6238 4850 50  0001 C CNN
 F 3 "~" H 6200 5000 50  0001 C CNN
 	1    6200 5000
@@
 Wire Wire Line
 	5850 4000 5850 4050
+$Comp
+L Connector:USB_B J1
+U 1 1 5C95669A
+P 2750 3200
+F 0 "J1" H 2805 3667 50  0000 C CNN
+F 1 "USB_B" H 2805 3576 50  0000 C CNN
+F 2 "Connector_USB:USB_B_OST_USB-B1HSxx_Horizontal" H 2900 3150 50  0001 C CNN
+F 3 " ~" H 2900 3150 50  0001 C CNN
+	1    2750 3200
+	1    0    0    -1
+$EndComp
 $EndSCHEMATC

Commit message: Placa 12V v0.9
Parts:
- C1: footprint Capacitor_THT:C_Disc_D5.0mm_W2.5mm_P2.50mm -> Capacitor_THT:C_Disc_D6.0mm_W2.5mm_P5.00mm
- RV1: footprint Potentiometer_THT:Potentiometer_Alps_RK09L_Single_Horizontal -> Potentiometer_THT:Potentiometer_Alps_RK163_Single_Horizontal
Changed lines of the file:
@@
 F 0 "C1" H 4415 3846 50  0000 L CNN
 F 1 "330nF" H 4415 3755 50  0000 L CNN
-F 2 "Capacitor_THT:C_Disc_D5.0mm_W2.5mm_P2.50mm" H 4338 3650 50  0001 C CNN
+F 2 "Capacitor_THT:C_Disc_D6.0mm_W2.5mm_P5.00mm" H 4338 3650 50  0001 C CNN
 F 3 "~" H 4300 3800 50  0001 C CNN
 	1    4300 3800
@@
 F 0 "RV1" H 5380 5396 50  0000 R CNN
 F 1 "5K" H 5380 5305 50  0000 R CNN
-F 2 "Potentiometer_THT:Potentiometer_Alps_RK09L_Single_Horizontal" H 5450 5350 50  0001 C CNN
+F 2 "Potentiometer_THT:Potentiometer_Alps_RK163_Single_Horizontal" H 5450 5350 50  0001 C CNN
 F 3 "~" H 5450 5350 50  0001 C CNN
 	1    5450 5350
